File: wearablesystem/wearablesystem.kicad_pcb (KiCad board)
At the start: 2 copper layers, 103 x 101.5 mm, 64 parts, among them J1 USB_C_Receptacle_USB2.0_16P, J2 Conn_01x04_Pin, J3 Conn_Coaxial, SW1 SW_Push, SW2 SW_Push, U1 ESP32-C3, U2 SPX3819M5-L-3-3, U3 SPX3819M5-L-1-8, U4 MAX30102, U5 W25Q16JVUXIQ TR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

Commit message: maybe fixed errors
Routing:
- net GND: track 231.4 -> 241.8 mm, vias 10 -> 13
- net +1V8: track 146.0 -> 154.8 mm
- net +3.3V: track 320.9 -> 318.8 mm
- net Net-(U1-GPIO8): track 14.9 -> 14.3 mm
- net /SDA: track 41.5 -> 40.9 mm

Commit message: added files plus gerber
Other:
- board text added: "Group 41 Ambient Lighting System Wearable System Version 3"
Changed lines of the file:
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@@
 		(layer "Edge.Cuts")
+	)
+	(gr_text "Group 41\nAmbient Lighting System\nWearable System\nVersion 3"
+		(at 104 114.5 0)
+		(layer "F.SilkS")
+		(effects
+			(font
+				(size 1 1)
+				(thickness 0.1)
+			)
+			(justify left bottom)
+		)
 	)
 	(dimension
@@
 		)
 		(height 0)
-		(gr_text "3.9695 in"
+		(gr_text "3969.4570 mils"
 			(at 74.965371 117.704229 0.003415326947)
 			(layer "F.Cu")
@@
 		)
 		(height 1.446644)
-		(gr_text "3.9371 in"
+		(gr_text "3937.0570 mils"
 			(at 26.103352 69.498233 270.2864765)
 			(layer "F.Cu")
@@
 		)
 		(height 0.122424)
-		(gr_text "3.9372 in"
+		(gr_text "3937.2047 mils"
 			(at 126.677492 69.483225 270.5729387)
 			(layer "F.Cu")
@@
 		)
 		(height 0)
-		(gr_text "3.9546 in"
+		(gr_text "3954.5916 mils"
 			(at 74.276557 17.703616 0.004126347343)
 			(layer "F.Cu")

Commit message: adding new files
Other:
- board size 103 x 101.5 mm -> 100.5 x 99.5 mm
Changed lines of the file:
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@@
 	(gr_rect
 		(start 24 19.5)
-		(end 127 121)
+		(end 124.5 119)
 		(stroke
 			(width 0.05)
