File: mounted_system/mounted_system.kicad_pcb (KiCad board)
At the start: 2 copper layers, 98.7 x 98.4 mm, 54 parts, among them J1 Conn_01x04_Pin, J2 Conn_Coaxial, J3 USB_C_Receptacle_USB2.0_16P, J4 Conn_01x05_Pin, J5 Conn_01x06_Pin, Q1 NMOS, Q2 NMOS, Q3 NMOS, SW1 SW_Push, SW2 SW_Push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

Commit message: maybe fixed errors
Routing:
- net GND: track 6.15 -> 42.8 mm, vias 21 -> 13
- net VBUS: track 88.3 -> 99.5 mm, vias 2 -> 4
- net /R: track 29.2 -> 40.0 mm
- net /USB_D-: track 35.6 -> 32.6 mm
- net /MICOUT: track 175.4 -> 176.6 mm
- net /G: track 22.4 -> 23.4 mm, vias 0 -> 1
- net /VDD_RF: track 50.4 -> 51.4 mm
- net /LED2: track 96.4 -> 95.5 mm
- net /VDD_BUSF: track 74.5 -> 75.1 mm, vias 6 -> 2
- net +3.3V: track 213.7 -> 213.9 mm, vias 18 -> 15
- net /B: track 22.8 -> 22.9 mm, vias 0 -> 1

Commit message: added files plus gerber
Routing:
- net GND: vias 13 -> 14
Other:
- board text added: "Group 41 Ambient Lighting System Mounted Subsystem Version 3"
Changed lines of the file:
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@@
 		(layer "Edge.Cuts")
+	)
+	(gr_text "Group 41\nAmbient Lighting System\nMounted Subsystem\nVersion 3"
+		(at 74 121 0)
+		(layer "F.SilkS")
+		(effects
+			(font
+				(size 1 1)
+				(thickness 0.1)
+			)
+			(justify left bottom)
+		)
 	)
 	(segment
@@
 		(size 0.6)
 		(drill 0.3)
+		(layers "F.Cu" "B.Cu")
+		(free yes)
+		(net 2)
+	)
+	(via
+		(at 115.5 64)
+		(size 0.6)
+		(drill 0.3)

Commit message: updated
Routing:
- net Net-(J3-D--PadA7): track 29.1 -> 25.3 mm
- net +3.3V: track 213.9 -> 214.4 mm, vias 15 -> 10
Changed lines of the file:
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@@
 		(tags "W25Q16JVUXIQ TR ")
 		(property "Reference" "U2"
-			(at 0 0 -90)
+			(at 0 2.83 -90)
 			(unlocked yes)
 			(layer "F.SilkS")
@@
 		)
 		(fp_text user "${REFERENCE}"
-			(at 0 0 -90)
+			(at 0 2.83 -90)
 			(unlocked yes)
 			(layer "F.Fab")
@@
 	)
 	(segment
-		(start 87.6785 49.8325)
-		(end 87.503 49.657)
-		(width 0.254)
-		(layer "F.Cu")
-		(net 6)
-	)
-	(segment
 		(start 81.153 56.769)
 		(end 81.153 57.428144)
@@
 	)
 	(segment
+		(start 88.362 49.149)
+		(end 88.011 49.149)
+		(width 0.254)
+		(layer "F.Cu")
+		(net 6)
+	)
+	(segment
 		(start 86.269 75.551)
 		(end 87.412 76.694)
@@
 	)
 	(segment
+		(start 90.17 65.748)
+		(end 90.17 66.675)
+		(width 0.254)
+		(layer "F.Cu")
+		(net 6)
+	)
+	(segment
 		(start 114.732 49.736)
 		(end 117.257 49.736)
@@
 	)
 	(segment
-		(start 90.17 66.675)
-		(end 90.17 65.748)
-		(width 0.254)
-		(layer "F.Cu")
-		(net 6)
-	)
-	(segment
 		(start 102.032 50.622)
 		(end 98.425 54.229)
@@
 	)
 	(segment
+		(start 102.032 49.8325)
+		(end 101.3485 49.149)
+		(width 0.254)
+		(layer "F.Cu")
+		(net 6)
+	)
+	(segment
 		(start 134.681 35.168)
 		(end 134.442 35.407)
@@
 	)
 	(segment
+		(start 88.011 49.149)
+		(end 87.884 49.276)
+		(width 0.254)
+		(layer "F.Cu")
+		(net 6)
+	)
+	(segment
 		(start 83.947 85.276)
 		(end 83.947 80.359)
@@
 	)
 	(segment
+		(start 83.635735 66.087978)
+		(end 84.153022 66.087978)
+		(width 0.2)
+		(layer "F.Cu")
+		(net 6)
+	)
+	(segment
 		(start 62.593 70.569)
 		(end 62.593 69.099)
@@
 	)
 	(segment
-		(start 102.032 49.8325)
-		(end 87.6785 49.8325)
+		(start 110.526 36.66)
+		(end 117.257 43.391)
 		(width 0.254)
 		(layer "F.Cu")
@@
 	)
 	(segment
-		(start 110.526 36.66)
-		(end 117.257 43.391)
+		(start 101.3485 49.149)
+		(end 88.362 49.149)
 		(width 0.254)
 		(layer "F.Cu")
@@
 	)
 	(segment
+		(start 84.153022 66.087978)
+		(end 84.201 66.04)
+		(width 0.2)
+		(layer "F.Cu")
+		(net 6)
+	)
+	(segment
 		(start 84.475 57.615)
 		(end 83.975 57.615)
@@
 	)
 	(via
-		(at 84.201 66.04)
-		(size 0.6)
-		(drill 0.3)
-		(layers "F.Cu" "B.Cu")
-		(net 6)
-	)
-	(via
-		(at 81.153 56.769)
-		(size 0.6)
-		(drill 0.3)
-		(layers "F.Cu" "B.Cu")
-		(net 6)
-	)
-	(via
 		(at 70.394 59.901)
 		(size 0.6)
@@
 	)
 	(via
-		(at 95.377 65.786)
-		(size 0.6)
-		(drill 0.3)
-		(layers "F.Cu" "B.Cu")
-		(net 6)
-	)
-	(via
-		(at 87.503 49.657)
-		(size 0.6)
-		(drill 0.3)
-		(layers "F.Cu" "B.Cu")
-		(net 6)
-	)
-	(via
 		(at 81.153 56.769)
 		(size 0.6)
@@
 	)
 	(via
-		(at 71.755 57.531)
+		(at 95.377 65.786)
 		(size 0.6)
 		(drill 0.3)
@@
 	)
 	(via
-		(at 84.201 66.04)
+		(at 83.635735 66.087978)
 		(size 0.6)
 		(drill 0.3)
@@
 	)
 	(via
-		(at 87.503 49.657)
-		(size 0.6)
-		(drill 0.3)
-		(layers "F.Cu" "B.Cu")
-		(net 6)
-	)
-	(via
-		(at 84.201 66.04)
+		(at 71.755 57.531)
 		(size 0.6)
 		(drill 0.3)
@@
 	)
 	(via
-		(at 90.17 66.675)
+		(at 87.884 49.276)
 		(size 0.6)
 		(drill 0.3)
@@
 	)
 	(segment
-		(start 79.121 57.428144)
-		(end 82.642 60.949144)
-		(width 0.2)
+		(start 69.251 62.441)
+		(end 69.251 61.044)
+		(width 0.254)
 		(layer "B.Cu")
 		(net 6)
 	)
 	(segment
-		(start 91.059 65.786)
-		(end 90.17 66.675)
+		(start 87.503 50.419)
+		(end 81.153 56.769)
 		(width 0.254)
 		(layer "B.Cu")
@@
 	)
 	(segment
-		(start 69.251 62.441)
-		(end 69.251 61.044)
+		(start 91.059 65.786)
+		(end 90.17 66.675)
 		(width 0.254)
 		(layer "B.Cu")
@@
 	)
 	(segment
-		(start 87.503 50.419)
-		(end 81.153 56.769)
+		(start 87.884 49.276)
+		(end 87.503 49.657)
 		(width 0.254)
 		(layer "B.Cu")
@@
 	)
 	(segment
-		(start 83.812471 66.04)
-		(end 84.201 66.04)
-		(width 0.2)
+		(start 79.780144 56.769)
+		(end 81.153 56.769)
+		(width 0.254)
 		(layer "B.Cu")
 		(net 6)
 	)
 	(segment
-		(start 82.642 60.949144)
-		(end 82.642 64.869529)
+		(start 71.857856 57.428144)
+		(end 79.121 57.428144)
 		(width 0.2)
 		(layer "B.Cu")
@@
 	)
 	(segment
-		(start 71.857856 57.428144)
-		(end 79.121 57.428144)
+		(start 82.642 65.116)
+		(end 83.613978 66.087978)
 		(width 0.2)
 		(layer "B.Cu")
@@
 	)
 	(segment
-		(start 71.755 57.531)
-		(end 71.857856 57.428144)
+		(start 79.121 57.428144)
+		(end 82.642 60.949144)
 		(width 0.2)
 		(layer "B.Cu")
@@
 	)
 	(segment
-		(start 82.642 64.869529)
-		(end 83.812471 66.04)
+		(start 71.755 57.531)
+		(end 71.857856 57.428144)
 		(width 0.2)
 		(layer "B.Cu")
@@
 	)
 	(segment
-		(start 81.153 56.769)
-		(end 79.780144 56.769)
-		(width 0.254)
+		(start 82.642 60.949144)
+		(end 82.642 65.116)
+		(width 0.2)
 		(layer "B.Cu")
 		(net 6)
 	)
 	(segment
-		(start 79.780144 56.769)
-		(end 79.121 57.428144)
-		(width 0.254)
+		(start 83.613978 66.087978)
+		(end 83.635735 66.087978)
+		(width 0.2)
 		(layer "B.Cu")
 		(net 6)
 	)
 	(segment
-		(start 69.251 61.044)
-		(end 70.394 59.901)
+		(start 79.780144 56.769)
+		(end 79.121 57.428144)
 		(width 0.254)
 		(layer "B.Cu")
@@
 	)
 	(segment
-		(start 90.043 66.802)
-		(end 90.17 66.675)
+		(start 69.251 61.044)
+		(end 70.394 59.901)
 		(width 0.254)
 		(layer "B.Cu")
@@
 	)
 	(segment
-		(start 112.352 70.823)
-		(end 112.141 70.612)
+		(start 114.717 71.918)
+		(end 116.332 73.533)
 		(width 0.2)
 		(layer "B.Cu")
@@
 	)
 	(segment
-		(start 113.622 70.823)
-		(end 112.352 70.823)
-		(width 0.2)
-		(layer "B.Cu")
-		(net 25)
-	)
-	(segment
-		(start 113.658 70.612)
-		(end 114.717 69.553)
-		(width 0.2)
-		(layer "B.Cu")
-		(net 25)
-	)
-	(segment
-		(start 112.141 70.612)
-		(end 113.658 70.612)
-		(width 0.2)
-		(layer "B.Cu")
-		(net 25)
-	)
-	(segment
-		(start 116.332 73.533)
-		(end 113.622 70.823)
+		(start 114.717 69.553)
+		(end 114.717 71.918)
 		(width 0.2)
 		(layer "B.Cu")
@@
 	)
 	(segment
-		(start 103.283 59.4668)
-		(end 102.9766 59.7732)
+		(start 101.727 60.325)
+		(end 99.187 57.785)
 		(width 0.254)
 		(layer "F.Cu")
@@
 	)
 	(segment
-		(start 99.187 57.785)
-		(end 93.891712 57.785)
+		(start 103.283 58.7794)
+		(end 103.283 59.4668)
 		(width 0.254)
 		(layer "F.Cu")
@@
 	)
 	(segment
-		(start 103.283 58.7794)
-		(end 103.283 59.4668)
+		(start 99.187 57.785)
+		(end 93.891712 57.785)
 		(width 0.254)
 		(layer "F.Cu")
@@
 	)
 	(segment
-		(start 101.8805 59.7732)
-		(end 101.8805 60.325)
+		(start 93.891712 57.785)
+		(end 93.361712 58.315)
 		(width 0.254)
 		(layer "F.Cu")
@@
 	)
 	(segment
-		(start 101.727 60.325)
-		(end 99.187 57.785)
+		(start 101.8805 60.325)
+		(end 101.727 60.325)
 		(width 0.254)
 		(layer "F.Cu")
@@
 	)
 	(segment
-		(start 93.891712 57.785)
-		(end 93.361712 58.315)
+		(start 103.283 59.4668)
+		(end 102.9766 59.7732)
 		(width 0.254)
 		(layer "F.Cu")
@@
 	)
 	(segment
-		(start 101.8805 60.325)
-		(end 101.727 60.325)
+		(start 101.8805 59.7732)
+		(end 101.8805 60.325)
 		(width 0.254)
 		(layer "F.Cu")
